Commit message: get rid of unknown material warning

File: talos_description/urdf/sensors/ftsensor.urdf.xacro (robot description, xacro)
@@ -43,5 +43,5 @@
           <cylinder radius="${0.05*0.5}" length="0.00975"/>
         </geometry>
-        <material name="FlatBlack" />
+        <!-- <material name="FlatBlack" /> -->
       </visual>
       <collision>
